File: hardware/control-board/inverter.kicad_sch (KiCad schematic)
At the start: 52 parts, among them Q2 C3M0021120D, Q3 C3M0021120D, Q4 C3M0021120D, Q5 C3M0021120D, U3 UCC21550, U4 UCC21550

Commit message: mcu controller added
Other:
- note added: "TODO: Fault lines???"
