File: hardware/control-board/tank.kicad_sch (KiCad schematic)
At the start: 0 parts

Commit message: added basic LC series resonant tank
Parts:
- added C8: C, symbol Device:C
- added L3: L, symbol Device:L
- added T1: 10:1, symbol Device:Transformer_1P_1S
- added T2: Current Transformer, symbol Device:Transformer_1P_1S
Connections:
- new net: L3.1, T1.4 (SB)
- new net: L3.2, T2.1 (AA)
- new net: C8.1, T1.3 (SA)
- new net: C8.2, T2.2 (AB)
- new net INVERTER_A: T1.1 (AA)
- new net INVERTER_B: T1.2 (AB)
Other:
- note added: "HIGH VOLTAGE"

Commit message: added titles to sheets
Other:
- title: (none) -> Resonant Tank
Changed lines of the file:
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@@
 	(generator_version "9.0")
 	(paper "A4")
+	(title_block
+		(title "Resonant Tank")
+	)
 	(text "HIGH VOLTAGE"
 		(exclude_from_sim no)

Commit message: reasearch, added section and finished negative bias addition to intervet side a
Connections:
- net INVERTER_A renamed SIDE_A
- net INVERTER_B renamed SIDE_B
Changed lines of the file:
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@@
 		)
 	)
-	(hierarchical_label "INVERTER_B"
+	(hierarchical_label "SIDE_B"
 		(shape input)
 		(at 93.98 104.14 180)
@@
 		)
 	)
-	(hierarchical_label "INVERTER_A"
+	(hierarchical_label "SIDE_A"
 		(shape input)
 		(at 93.98 93.98 180)
